File: rpi-cm4-xenon-carrier/cm4-gpio.kicad_sch (KiCad schematic)
At the start: 1 part

Commit message: update
Parts:
- added CR?: SMBJ5.0A-TR, SMB_STM, symbol SMBJ5.0A-TR:SMBJ5.0A-TR
- added J?: USB4105_REVA, GCT_USB4105_REVA, symbol USB4105_REVA:USB4105_REVA
Connections:
- new net: J?.A1/B12 (GND), J?.B1/A12 (GND), J?.G1 (GND), J?.G2 (GND), J?.G3 (GND), J?.G4 (GND)
- new net: J?.A4/B9 (VBUS), J?.B4/A9 (VBUS)
Changed lines of the file:
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@@
     (pin "1")
+  )
+  (symbol (lib_id "SMBJ5.0A-TR:SMBJ5.0A-TR") (at 181.61 81.28 0) (unit 1)
+    (in_bom yes) (on_board yes) (fields_autoplaced)
+    (property "Reference" "CR?" (id 0) (at 186.69 73.66 0)
+      (effects (font (size 1.524 1.524)))
+    )
+    (property "Value" "SMBJ5.0A-TR" (id 1) (at 186.69 77.47 0)
+      (effects (font (size 1.524 1.524)))
+    )
+    (property "Footprint" "SMB_STM" (id 2) (at 182.88 87.249 0)
+      (effects (font (size 1.524 1.524)) hide)
+    )
+    (property "Datasheet" "" (id 3) (at 181.61 81.28 0)
+      (effects (font (size 1.524 1.524)))
+    )
+    (pin "1")
+    (pin "2")
+  )
+  (symbol (lib_id "USB4105_REVA:USB4105_REVA") (at 180.34 45.72 0) (unit 1)
+    (in_bom yes) (on_board yes) (fields_autoplaced)
+    (property "Reference" "J?" (id 0) (at 180.34 27.94 0))
+    (property "Value" "USB4105_REVA" (id 1) (at 180.34 30.48 0))
+    (property "Footprint" "GCT_USB4105_REVA" (id 2) (at 180.34 45.72 0)
+      (effects (font (size 1.27 1.27)) (justify left bottom) hide)
+    )
+    (property "Datasheet" "" (id 3) (at 180.34 45.72 0)
+      (effects (font (size 1.27 1.27)) (justify left bottom) hide)
+    )
+    (property "PARTREV" "0.2" (id 4) (at 180.34 45.72 0)
+      (effects (font (size 1.27 1.27)) (justify left bottom) hide)
+    )
+    (property "STANDARD" "Manufacturer Recommendations" (id 5) (at 180.34 45.72 0)
+      (effects (font (size 1.27 1.27)) (justify left bottom) hide)
+    )
+    (property "MAXIMUM_PACKAGE_HEIGHT" "3.31 mm" (id 6) (at 180.34 45.72 0)
+      (effects (font (size 1.27 1.27)) (justify left bottom) hide)
+    )
+    (property "MANUFACTURER" "GCT" (id 7) (at 180.34 45.72 0)
+      (effects (font (size 1.27 1.27)) (justify left bottom) hide)
+    )
+    (pin "A1/B12")
+    (pin "A4/B9")
+    (pin "A5")
+    (pin "A6")
+    (pin "A7")
+    (pin "A8")
+    (pin "B1/A12")
+    (pin "B4/A9")
+    (pin "B5")
+    (pin "B6")
+    (pin "B7")
+    (pin "B8")
+    (pin "G1")
+    (pin "G2")
+    (pin "G3")
+    (pin "G4")
   )
   (symbol (lib_id "CM4IO:ComputeModule4-CM4") (at 76.2 101.6 0) (unit 1)
