File: rpi-cm4-xenon-carrier/cm4-gpio.kicad_sch (KiCad schematic)
At the start: 3 parts

Commit message: Update
Parts:
- removed CR?: SMBJ5.0A-TR, SMB_STM, symbol SMBJ5.0A-TR:SMBJ5.0A-TR
- added CR?: SMBJ5.0A-TR, SMBJ5.0A-TR:SMBJ5.0A-TR, symbol SMBJ5.0A-TR:SMBJ5.0A-TR
- added Q? (x5): 2N2219, Package_TO_SOT_THT:TO-39-3, symbol Transistor_BJT:2N2219
- added R? (x4): 10K, symbol Device:R
- added R? (x2): 5K, symbol Device:R
- added R? (x2): 5.1k, symbol Device:R
- added R? (x2): R, symbol Device:R
- added SW?: SW_Push_Power, symbol Switch:SW_Push
- added SW?: SW_DIP_x01, symbol Switch:SW_DIP_x01
- J?: footprint GCT_USB4105_REVA -> USB4105_REVA:GCT_USB4105_REVA; Digi-key_PN (none) -> 2073-USB4105-GF-ACT-ND; MPN (none) -> USB4105-GF-A
Connections:
- net +1.8V: now also SW?.1
- net +5V: now also J?.A4/B9 (VBUS), J?.B4/A9 (VBUS), CR?.1
- net GND: now also J?.A1/B12 (GND), J?.B1/A12 (GND), J?.G1 (GND), J?.G2 (GND), J?.G3 (GND), J?.G4 (GND), CR?.2, Q?.1 (E), R?.2, R?.2, R?.2, R?.2
- net at J?.A5 (CC1): now also R?.1
- net at J?.B5 (CC2): now also R?.1
- new net: R?.1, R?.1, SW?.2
- new net: Q?.2 (B), R?.2 (x4)
- new net: Q?.1 (E), R?.1 (x2)
- new net: Q?.1 (E), Q?.3 (C) (x2)
- new net: R?.1, R?.2, SW?.2
- new net: Q?.3 (C), R?.1, R?.1
- new net: Q?.2 (B), R?.1
- new net VCC: Q?.3 (C), Q?.3 (C), R?.2

Commit message: waaaay updated
Parts:
- removed SW?: SW_DIP_x01, symbol Switch:SW_DIP_x01
- added J?: Conn_01x05_Female, symbol Connector:Conn_01x05_Female
- added R?: 10K, symbol Device:R
- added R?: 1K, symbol Device:R
Connections:
- net VCC is gone; now on net +3.3V: Q?.3 (C), Q?.3 (C), R?.2
- net +1.8V: no longer SW?.1
- net +3.3V: now also SW?.1
- net GND: now also J?.5 (Pin_5), R?.1
- net at Q?.1 (E), R?.1: now also R?.1, R?.2
- net GPIO_PIN_22: now reaches Module1.46 (GPIO22)
- net GPIO_PIN_27: now reaches Module1.48 (GPIO27)
- net GPIO_PIN_27: now also R?.1, R?.2, R?.2
- net GPIO_PIN_17: now reaches Module1.50 (GPIO17)
- net RUN_PIN: now reaches Module1.92 (RUN_PG)
- net RUN_PIN: now also Q?.1 (E), R?.1
Other:
- note added: "3.3v"
- note added: "I belive this is a pullup resistor"
- note added: "The GPIO pins supply 3.3v by default"
- note added: "The resistance of these transistors is still up for debate, this resistance might not actually work at all, because electricity wants to flow where its easiest, but the resistor is kind of required"
- moved on the sheet: Q?, R?, SW?

Commit message: RP2040
Parts:
- removed Q? (x5): 2N2219, Package_TO_SOT_THT:TO-39-3, symbol Transistor_BJT:2N2219
- removed R? (x5): 10K, symbol Device:R
- removed R? (x2): 5K, symbol Device:R
- removed R? (x2): R, symbol Device:R
- removed R?: 1K, symbol Device:R
- removed SW?: SW_Push_Power, symbol Switch:SW_Push
Other:
- added sheet PowerButton (powerbutton.kicad_sch)
- added sheet SkittleChip (skittlechip.kicad_sch)
- note removed: "I belive this is a pullup resistor"
- note removed: "The GPIO pins supply 3.3v by default"
- note removed: "The resistance of these transistors is still up for debate, this resistance might not actually work at all, because electricity wants to flow where its easiest, but the resistor is kind of required"
- moved on the sheet: J?
