File: rpi-cm4-xenon-carrier/rpi-cm4-xenon-carrier.kicad_pcb (KiCad board)
At the start: 2 copper layers, 40 x 55 mm, 1 part

Commit message: waaaay updated
Other:
- board text added: "77Z Lichtgeschwindigkeit Approved by: Vince"
